File: kicad/rasp.sch (KiCad schematic (older format))
At the start: 18 parts, among them J1 RJ45, J2 RJ45, J3 RJ45, J4 RJ45, J5 RJ45, J6 RJ45, P1 CONN_01X01, P2 CONN_01X01, P3 CONN_01X01, P4 CONN_01X01, P5 DIL_26, U1 ULN2003A, U2 7805

Commit message: pins infos
Other:
- note added: "PIN 17"
- note added: "PIN 27"
- note added: "PIN 9"
Changed lines of the file:
@@
 LIBS:contrib
 LIBS:valves
+LIBS:rasp-cache
 EELAYER 25 0
 EELAYER END
@@
 Connection ~ 5550 4350
 Connection ~ 5400 5450
-Wire Wire Line
-	4700 5450 5400 5450
 NoConn ~ 3800 1850
 NoConn ~ 3800 1950
@@
 $EndComp
 NoConn ~ 1550 5000
+Text Notes 6850 3550 0    60   ~ 0
+PIN 9
+Text Notes 6900 2350 0    60   ~ 0
+PIN 27
+Text Notes 6900 1100 0    60   ~ 0
+PIN 17
 $EndSCHEMATC
